Commit message: firebase

File: install/linorobot2_description/share/linorobot2_description/urdf/6wd_properties.urdf.xacro (robot description, xacro)
@@ -13,5 +13,5 @@
   <xacro:property name="wheel_pos_y_2" value="0.06775" />
   <xacro:property name="wheel_pos_z" value="-0.04788" />
-  <xacro:property name="wheel_mass" value=".6" />
+  <xacro:property name="wheel_mass" value="0.6" />
   <xacro:property name="wheel_torque" value="20" />
   <xacro:property name="laser_pose">

File: install/linorobot2_description/share/linorobot2_description/urdf/robots/6wd.urdf.xacro (robot description, xacro)
@@ -49,5 +49,5 @@
     width="${wheel_width}"
     pos_x="${wheel_pos_x_2}"
-    pos_y="${-wheel_pos_y_2}"
+    pos_y="${wheel_pos_y_2}"
     pos_z="${wheel_pos_z}"
     mass="${wheel_mass}"
